Commit message: Fix: aggiornata compatibilità MoveIt2 e ros2_control per ROS 2 Jazzy

File: myco_10_1000mm/myco_10_1000mm_ros2_moveit2/config/MyCo-10-1.00.ros2_control.xacro (robot description, xacro)
@@ -1,5 +1,5 @@
 <?xml version="1.0"?>
 <robot xmlns:xacro="http://www.ros.org/wiki/xacro">
-    <xacro:macro name="MyCo-10-1.00_ros2_control" params="name initial_positions_file">
+    <xacro:macro name="MyCo-10-1_00_ros2_control" params="name initial_positions_file">
         <xacro:property name="initial_positions" value="${load_yaml(initial_positions_file)['initial_positions']}"/>
         <ros2_control name="${name}" type="system">

File: myco_10_1000mm/myco_10_1000mm_ros2_moveit2/config/MyCo-10-1.00.urdf.xacro (robot description, xacro)
@@ -6,4 +6,4 @@
     <!-- Import control_xacro -->
     <xacro:include filename="MyCo-10-1.00.ros2_control.xacro" />
-    <xacro:MyCo-10-1.00_ros2_control name="FakeSystem" initial_positions_file="$(arg initial_positions_file)"/>
+    <xacro:MyCo-10-1_00_ros2_control name="FakeSystem" initial_positions_file="$(arg initial_positions_file)"/>
 </robot>
